File: electronics/_autosave-miniclick.kicad_sch (KiCad schematic)
At the start: 25 parts, among them J1 Stemma QT, J2 Stemma QT, J4 Joystick Mount, SW1 SW_MEC_5E, SW2 SW_MEC_5E, SW3 SW_MEC_5E, SW5 SW_MEC_5E, U1 ATSAMD09D14A-M

Commit message: pcb V2
Connections:
- net PA4 is gone; now on net PA6: SW1.4 (A), U1.5 (PA06)
- net GND: now also U1.23 (GND)
- net LED: now also R3.1, U1.8 (PA09/XOUT)
- net PA6: no longer SW3.4 (A), U1.7 (PA08/XIN)
- net PA11: now reaches U1.10 (PA11)
- net PA11: now also SW5.4 (A)
- net PA8: now reaches U1.7 (PA08/XIN)
- net PA8: now also SW3.4 (A)
- removed net PA2: SW5.4 (A), U1.8 (PA09/XOUT)
- net PA5 renamed PA7
Changed lines of the file:
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@@
     )
   )
-  (global_label "PA6" (shape input) (at 67.31 63.5 90) (fields_autoplaced)
+  (global_label "PA8" (shape input) (at 67.31 63.5 90) (fields_autoplaced)
     (effects (font (size 1.27 1.27)) (justify left))
     (property "Intersheetrefs" "${INTERSHEET_REFS}" (at 67.31 56.9467 90)
@@
     )
   )
-  (global_label "PA4" (shape input) (at 36.83 63.5 90) (fields_autoplaced)
+  (global_label "PA6" (shape input) (at 36.83 63.5 90) (fields_autoplaced)
     (effects (font (size 1.27 1.27)) (justify left))
     (property "Intersheetrefs" "${INTERSHEET_REFS}" (at 36.83 56.9467 90)
@@
     )
   )
-  (global_label "PA2" (shape input) (at 21.59 63.5 90) (fields_autoplaced)
-    (effects (font (size 1.27 1.27)) (justify left))
-    (property "Intersheetrefs" "${INTERSHEET_REFS}" (at 21.59 56.9467 90)
+  (global_label "PA11" (shape input) (at 21.59 63.5 90) (fields_autoplaced)
+    (effects (font (size 1.27 1.27)) (justify left))
+    (property "Intersheetrefs" "${INTERSHEET_REFS}" (at 21.59 55.7372 90)
       (effects (font (size 1.27 1.27)) (justify left) hide)
     )
@@
     )
   )
-  (global_label "LED" (shape input) (at 156.21 80.01 0) (fields_autoplaced)
-    (effects (font (size 1.27 1.27)) (justify left))
-    (property "Intersheetrefs" "${INTERSHEET_REFS}" (at 162.6423 80.01 0)
+  (global_label "LED" (shape input) (at 153.67 93.98 0) (fields_autoplaced)
+    (effects (font (size 1.27 1.27)) (justify left))
+    (property "Intersheetrefs" "${INTERSHEET_REFS}" (at 160.1023 93.98 0)
       (effects (font (size 1.27 1.27)) (justify left) hide)
     )
@@
     )
   )
-  (global_label "PA2" (shape input) (at 153.67 93.98 0) (fields_autoplaced)
-    (effects (font (size 1.27 1.27)) (justify left))
-    (property "Intersheetrefs" "${INTERSHEET_REFS}" (at 160.2233 93.98 0)
+  (global_label "PA11" (shape input) (at 153.67 99.06 0) (fields_autoplaced)
+    (effects (font (size 1.27 1.27)) (justify left))
+    (property "Intersheetrefs" "${INTERSHEET_REFS}" (at 161.4328 99.06 0)
+      (effects (font (size 1.27 1.27)) (justify left) hide)
+    )
+  )
+  (global_label "LED" (shape input) (at 83.82 99.06 90) (fields_autoplaced)
+    (effects (font (size 1.27 1.27)) (justify left))
+    (property "Intersheetrefs" "${INTERSHEET_REFS}" (at 83.82 92.6277 90)
       (effects (font (size 1.27 1.27)) (justify left) hide)
     )
@@
     )
   )
-  (global_label "PA5" (shape input) (at 50.8 63.5 90) (fields_autoplaced)
+  (global_label "PA7" (shape input) (at 50.8 63.5 90) (fields_autoplaced)
     (effects (font (size 1.27 1.27)) (justify left))
     (property "Intersheetrefs" "${INTERSHEET_REFS}" (at 50.8 56.9467 90)
@@
     )
   )
-  (global_label "PA5" (shape input) (at 153.67 88.9 0) (fields_autoplaced)
+  (global_label "PA7" (shape input) (at 153.67 88.9 0) (fields_autoplaced)
     (effects (font (size 1.27 1.27)) (justify left))
     (property "Intersheetrefs" "${INTERSHEET_REFS}" (at 160.2233 88.9 0)
@@
     )
   )
-  (global_label "PA4" (shape input) (at 153.67 86.36 0) (fields_autoplaced)
+  (global_label "PA6" (shape input) (at 153.67 86.36 0) (fields_autoplaced)
     (effects (font (size 1.27 1.27)) (justify left))
     (property "Intersheetrefs" "${INTERSHEET_REFS}" (at 160.2233 86.36 0)
@@
     )
   )
-  (global_label "PA6" (shape input) (at 153.67 91.44 0) (fields_autoplaced)
+  (global_label "PA8" (shape input) (at 153.67 91.44 0) (fields_autoplaced)
     (effects (font (size 1.27 1.27)) (justify left))
     (property "Intersheetrefs" "${INTERSHEET_REFS}" (at 160.2233 91.44 0)
@@
     )
   )
-  (symbol (lib_id "power:GND") (at 140.97 121.92 0) (unit 1)
-    (in_bom yes) (on_board yes) (dnp no) (fields_autoplaced)
-    (property "Reference" "#PWR013" (at 140.97 128.27 0)
-      (effects (font (size 1.27 1.27)) hide)
-    )
-    (property "Value" "GND" (at 140.97 127 0)
-      (effects (font (size 1.27 1.27)))
-    )
-    (property "Footprint" "" (at 140.97 121.92 0)
-      (effects (font (size 1.27 1.27)) hide)
-    )
-    (property "Datasheet" "" (at 140.97 121.92 0)
-      (effects (font (size 1.27 1.27)) hide)
-    )
+  (symbol (lib_id "power:GND") (at 140.97 125.73 0) (unit 1)
+    (in_bom yes) (on_board yes) (dnp no) (fields_autoplaced)
+    (property "Reference" "#PWR013" (at 140.97 132.08 0)
+      (effects (font (size 1.27 1.27)) hide)
+    )
+    (property "Value" "GND" (at 140.97 130.81 0)
+      (effects (font (size 1.27 1.27)))
+    )
+    (property "Footprint" "" (at 140.97 125.73 0)
+      (effects (font (size 1.27 1.27)) hide)
+    )
+    (property "Datasheet" "" (at 140.97 125.73 0)
+      (effects (font (size 1.27 1.27)) hide)
+    )
