File: electronics/miniclick.kicad_pcb (KiCad board)
At the start: 4 copper layers, 20 x 29 mm, 24 parts, among them J1 Stemma QT, J2 Stemma QT, J3 JTAG, J4 Joystick Mount, SW1 SW_MEC_5E, SW2 SW_MEC_5E, SW3 SW_MEC_5E, SW5 SW_MEC_5E, U1 ATSAMD09D14A-M

Commit message: pcb V2
Parts:
- removed J3: JTAG, Connector_PinHeader_1.27mm:PinHeader_2x05_P1.27mm_Vertical_SMD
- added D6: LED, LED_SMD:LED_0805_2012Metric, B.Cu at (141.6, 93.1)
- added R3: 10k, Resistor_SMD:R_0402_1005Metric, B.Cu at (141.6, 90.2)
- J4: footprint Connector_PinHeader_1.00mm:PinHeader_1x01_P1.00mm_Vertical -> Connector_PinHeader_2.00mm:PinHeader_1x01_P2.00mm_Vertical
- R1: value 10k -> locked
- TP1: value TestPoint -> nRST
- moved R1 2.19 mm to (139.4, 90.2)
- moved D1 2.10 mm to (139.5, 93.1)
- turned J4 to 180 degrees
Connections:
- net /nRST renamed nRST
- SW1 pad 4: PA3 -> PA4
- SW2 pad 4: PA4 -> PA5
- SW3 pad 4: PA5 -> PA6
- U1 pad 3: PA3 -> unconnected-(U1-PA04-Pad3)
- U1 pad 4: PA4 -> unconnected-(U1-PA05-Pad4)
- U1 pad 5: PA5 -> PA4
- U1 pad 6: unconnected-(U1-PA07-Pad6) -> PA5
- U1 pad 7: unconnected-(U1-PA08/XIN-Pad7) -> PA6
- U1 pad 8: unconnected-(U1-PA09/XOUT-Pad8) -> LED
Routing:
- net PA5: track 4.19 -> 25.3 mm, vias 1 -> 3
- net SWDCLK: track 25.5 -> 4.75 mm, vias 2 -> 0
- net SWDIO: track 26.6 -> 5.93 mm, vias 2 -> 0
- net PA3: track 14.3 -> 0.00 mm, vias 1 -> 0
- net nRST: track 15.9 -> 5.35 mm
- net PA4: track 24.9 -> 15.2 mm, vias 3 -> 1
- net GND: track 46.9 -> 40.9 mm, vias 17 -> 16
- net PA6: track 0.00 -> 5.18 mm, vias 0 -> 1
- net LED: track 0.00 -> 4.28 mm
- net +3.3V: track 20.7 -> 18.5 mm, vias 11 -> 9
- net Net-(D6-A): track 0.00 -> 2.17 mm
- net unconnected-(SW5-Pad2): track 0.00 -> 1.32 mm
- net SDA: track 38.6 -> 37.4 mm
- net PA2: track 4.96 -> 6.12 mm
- net SCL: track 44.3 -> 43.8 mm
Other:
- board size 20 x 29 mm -> 20 x 20 mm
